File: Dual Axis Tracker/hardware/Arduino-Nano-Board/Arduino-Nano-Board.kicad_pcb (KiCad board)
At the start: 2 copper layers, 54.6 x 48.3 mm, 12 parts, among them J1 SERVO, J2 SERVO, J3 TO LDR BOARD, M3 HOLE-PLATED-3.6MM, U1 ARDUINO-NANO

Commit message: Update to v1.5, number change only
Other:
- board text added: "Solar Tracker Nano Shield v1.5 Brown Dog Gadgets"
- board text removed: "Solar Tracker Nano Shield v1.0 Brown Dog Gadgets"
Changed lines of the file:
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@@
     (links 22)
     (no_connects 1)
-    (area 15.163799 45.643799 69.926201 94.056201)
+    (area 11.923143 23.3934 222.753159 94.056201)
     (thickness 1.6)
     (drawings 34)
@@
     (title "Solar Tracker Arduino Nano Board")
     (date "12 Mar 2018")
-    (rev 1.0)
+    (rev "v1.5")
     (company "All rights reserved.")
-    (comment 1 help@browndoggadgets.com)
-    (comment 2 http://browndoggadgets.com/)
+    (comment 1 "help@browndoggadgets.com")
+    (comment 2 "http://browndoggadgets.com/")
     (comment 3 "Brown Dog Gadgets")
   )
@@
   )
   (setup
-    (last_trace_width 0.762)
+    (last_trace_width 0.254)
     (user_trace_width 0.1524)
     (user_trace_width 0.254)
@@
   (gr_line (start 69.85 52.07) (end 69.85 87.63) (layer Edge.Cuts) (width 0.1524))
   (gr_arc (start 63.5 52.07) (end 63.5 45.72) (angle 90) (layer Edge.Cuts) (width 0.1524))
-  (gr_text "Solar Tracker Nano Shield v1.0\n\nBrown Dog Gadgets" (at 39.0398 67.5132 90) (layer B.SilkS)
+  (gr_text "Solar Tracker Nano Shield v1.5\n\nBrown Dog Gadgets" (at 39.0398 67.5132 90) (layer B.SilkS)
     (effects (font (size 1.5 1.5) (thickness 0.3)) (justify mirror))
   )
