File: Dual Axis Tracker/hardware/LDR-Board/LDR-Board.kicad_pcb (KiCad board)
At the start: 2 copper layers, 29.2 x 40.6 mm, 7 parts, among them J1 TO SOLAR SHIELD

Commit message: change version on silk
Other:
- board text added: "LDR Board v1.3.2"
- board text removed: "LDR Board v1.3"
Changed lines of the file:
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@@
-      (effects (font (size 1 1) (thickness 0.15)))
-    )
-    (fp_text user BR (at 0 -3.81 90) (layer F.SilkS)
       (effects (font (size 1 1) (thickness 0.15)))
     )
@@
     (effects (font (size 1.5 1.5) (thickness 0.3)) (justify mirror))
   )
-  (gr_text "LDR Board v1.3\n" (at 6.985 64.77 90) (layer B.SilkS)
+  (gr_text "LDR Board v1.3.2\n" (at 6.985 64.77 90) (layer B.SilkS)
     (effects (font (size 1.5 1.5) (thickness 0.3)) (justify mirror))
   )
